File: hardware/connection-board-cut-out_3_5/connection-board-cut-out_3_5.kicad_pcb (KiCad board)
At the start: 2 copper layers, 175 x 90 mm, 28 parts

Commit message: docs(hardware): label pcb variants on silkscreen
Add clear variant labels to the board version line so the two
connector board variants can be identified directly on the PCB.

Made-with: Cursor
Other:
- board text added: "Open Locker Connector Board Version: 1.1.0 (Terminal Block 3.50 mm) Power supply: 12V Bus: Modbus RTU Docs: https://github.com/Open-Locker/Open-Locker Designed for: https://www.waveshare.com/wiki/Modbus_RTU_Relay_(D)"
- board text removed: "Open Locker Connector Board Version: 1.1.0 Power supply: 12V Bus: Modbus RTU Docs: https://github.com/Open-Locker/Open-Locker Designed for: https://www.waveshare.com/wiki/Modbus_RTU_Relay_(D)"
Changed lines of the file:
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@@
 		)
 	)
-	(gr_text "Open Locker Connector Board\n\nVersion: 1.1.0\n\nPower supply: 12V\nBus: Modbus RTU\n\nDocs: https://github.com/Open-Locker/Open-Locker\nDesigned for: https://www.waveshare.com/wiki/Modbus_RTU_Relay_(D)"
+	(gr_text "Open Locker Connector Board\n\nVersion: 1.1.0 (Terminal Block 3.50 mm)\n\nPower supply: 12V\nBus: Modbus RTU\n\nDocs: https://github.com/Open-Locker/Open-Locker\nDesigned for: https://www.waveshare.com/wiki/Modbus_RTU_Relay_(D)"
 		(at 219 122 90)
 		(layer "F.SilkS")

Commit message: add 1N4007 diode between power supply and coil
Parts:
- added D1: 1N4007, Diode_THT:D_DO-41_SOD81_P10.16mm_Horizontal, F.Cu at (91.7, 81.8)
- added D2: 1N4007, Diode_THT:D_DO-41_SOD81_P10.16mm_Horizontal, F.Cu at (107.1, 81.8)
- added D3: 1N4007, Diode_THT:D_DO-41_SOD81_P10.16mm_Horizontal, F.Cu at (122.2, 81.8)
- added D4: 1N4007, Diode_THT:D_DO-41_SOD81_P10.16mm_Horizontal, F.Cu at (137.5, 81.8)
- added D5: 1N4007, Diode_THT:D_DO-41_SOD81_P10.16mm_Horizontal, F.Cu at (152.9, 81.8)
- added D6: 1N4007, Diode_THT:D_DO-41_SOD81_P10.16mm_Horizontal, F.Cu at (168.3, 81.8)
- added D7: 1N4007, Diode_THT:D_DO-41_SOD81_P10.16mm_Horizontal, F.Cu at (183.6, 81.8)
- added D8: 1N4007, Diode_THT:D_DO-41_SOD81_P10.16mm_Horizontal, F.Cu at (199.0, 81.8)
Connections:
- LOCK_1 pad 1: Net-(CH_1-Pin_2) -> Net-(D1-K)
- LOCK_2 pad 1: Net-(CH_2-Pin_2) -> Net-(D2-K)
- LOCK_3 pad 1: Net-(CH_3-Pin_2) -> Net-(D3-K)
- LOCK_4 pad 1: Net-(CH_4-Pin_2) -> Net-(D4-K)
- LOCK_5 pad 1: Net-(CH_5-Pin_2) -> Net-(D5-K)
- LOCK_6 pad 1: Net-(CH_6-Pin_2) -> Net-(D6-K)
- LOCK_7 pad 1: Net-(CH_7-Pin_2) -> Net-(D7-K)
- LOCK_8 pad 1: Net-(CH_8-Pin_2) -> Net-(D8-K)
Routing:
- net Net-(D1-K): track 0.00 -> 10.3 mm
- net Net-(D8-K): track 0.00 -> 9.55 mm
- net Net-(D2-K): track 0.00 -> 9.33 mm
- net Net-(D7-K): track 0.00 -> 8.85 mm
- net Net-(D6-K): track 0.00 -> 8.85 mm
- net Net-(D5-K): track 0.00 -> 8.85 mm
- net Net-(D4-K): track 0.00 -> 8.85 mm
- net Net-(D3-K): track 0.00 -> 8.85 mm
- net Net-(CH_2-Pin_2): track 14.7 -> 8.22 mm
- net Net-(CH_6-Pin_2): track 14.0 -> 8.48 mm
- net Net-(CH_3-Pin_2): track 14.0 -> 8.48 mm
- net Net-(CH_7-Pin_2): track 14.0 -> 8.48 mm
- net Net-(CH_5-Pin_2): track 14.0 -> 8.48 mm
- net Net-(CH_4-Pin_2): track 14.0 -> 8.48 mm
- net Net-(CH_8-Pin_2): track 14.0 -> 8.50 mm
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Other:
- board text added: "Open Locker Connector Board Version: 1.2.0 (Terminal Block 3.50 mm) Power supply: 12V Bus: Modbus RTU Docs: https://github.com/Open-Locker/Open-Locker Designed for: https://www.waveshare.com/wiki/Modbus_RTU_Relay_(D)"
- board text removed: "Open Locker Connector Board Version: 1.1.0 (Terminal Block 3.50 mm) Power supply: 12V Bus: Modbus RTU Docs: https://github.com/Open-Locker/Open-Locker Designed for: https://www.waveshare.com/wiki/Modbus_RTU_Relay_(D)"
