File: hardware/connection-board-cut-out_3_5/connection-board-cut-out_3_5.kicad_pcb (KiCad board)
At the start: 2 copper layers, 175 x 90 mm, 36 parts

Commit message: style(pcb): clarify 12V silkscreen polarity
Co-authored-by: Cursor <cursoragent@cursor.com>
Other:
- board text added: "+12V"
- board text added: "+12V Main power supply"
- board text added: "Open Locker Connector Board Version: 1.2.0 (Terminal Block 3.50 mm) Power supply: +12V Bus: Modbus RTU Docs: https://github.com/Open-Locker/Open-Locker Designed for: https://www.waveshare.com/wiki/Modbus_RTU_Relay_(D)"
- board text removed: "12V"
- board text removed: "12V Main power supply"
- board text removed: "Open Locker Connector Board Version: 1.2.0 (Terminal Block 3.50 mm) Power supply: 12V Bus: Modbus RTU Docs: https://github.com/Open-Locker/Open-Locker Designed for: https://www.waveshare.com/wiki/Modbus_RTU_Relay_(D)"
Changed lines of the file:
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@@
 		(layer "Edge.Cuts")
 	)
-	(gr_text "12V"
+	(gr_text "+12V"
 		(at 76 118.472 0)
 		(layer "F.SilkS")
@@
 		)
 	)
-	(gr_text "12V"
+	(gr_text "+12V"
 		(at 92.085714 118.472 0)
 		(layer "F.SilkS")
@@
 		)
 	)
-	(gr_text "12V"
+	(gr_text "+12V"
 		(at 107.185714 118.472 0)
 		(layer "F.SilkS")
@@
 		)
 	)
-	(gr_text "12V"
+	(gr_text "+12V"
 		(at 122.190357 118.472 0)
 		(layer "F.SilkS")
@@
 		)
 	)
-	(gr_text "12V"
+	(gr_text "+12V"
 		(at 137.785714 118.572 0)
 		(layer "F.SilkS")
@@
 		)
 	)
-	(gr_text "12V Main \npower supply\n"
+	(gr_text "+12V Main \npower supply\n"
 		(at 83.9 112.7 0)
 		(layer "F.SilkS")
@@
 		)
 	)
-	(gr_text "Open Locker Connector Board\n\nVersion: 1.2.0 (Terminal Block 3.50 mm)\n\nPower supply: 12V\nBus: Modbus RTU\n\nDocs: https://github.com/Open-Locker/Open-Locker\nDesigned for: https://www.waveshare.com/wiki/Modbus_RTU_Relay_(D)"
+	(gr_text "Open Locker Connector Board\n\nVersion: 1.2.0 (Terminal Block 3.50 mm)\n\nPower supply: +12V\nBus: Modbus RTU\n\nDocs: https://github.com/Open-Locker/Open-Locker\nDesigned for: https://www.waveshare.com/wiki/Modbus_RTU_Relay_(D)"
 		(at 219 122 90)
 		(layer "F.SilkS")
