File: hardware/mtu-connection-board/locker.kicad_pcb (KiCad board)
At the start: 2 copper layers, 112 x 72 mm, 22 parts

Commit message: style(pcb): clarify 12V silkscreen polarity
Co-authored-by: Cursor <cursoragent@cursor.com>
Other:
- board text added: "+12V"
- board text removed: "12V"
Changed lines of the file:
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@@
 		)
 	)
-	(gr_text "12V"
+	(gr_text "+12V"
 		(at 138 65.5 0)
 		(layer "F.SilkS")
@@
 		)
 	)
-	(gr_text "12V"
+	(gr_text "+12V"
 		(at 80 99.5 270)
 		(layer "F.SilkS")
@@
 		)
 	)
-	(gr_text "12V"
+	(gr_text "+12V"
 		(at 97.5 65.5 0)
 		(layer "F.SilkS")
@@
 		)
 	)
-	(gr_text "12V"
+	(gr_text "+12V"
 		(at 53 99.5 270)
 		(layer "F.SilkS")
@@
 		)
 	)
-	(gr_text "12V"
+	(gr_text "+12V"
 		(at 129 100 270)
 		(layer "F.SilkS")
@@
 		)
 	)
-	(gr_text "12V"
+	(gr_text "+12V"
 		(at 84 65.5 0)
 		(layer "F.SilkS")
@@
 		)
 	)
-	(gr_text "12V"
+	(gr_text "+12V"
 		(at 42 99.5 270)
 		(layer "F.SilkS")
@@
 		)
 	)
-	(gr_text "12V"
+	(gr_text "+12V"
 		(at 92.5 99.5 270)
 		(layer "F.SilkS")
@@
 		)
 	)
-	(gr_text "12V"
+	(gr_text "+12V"
 		(at 70.5 65.5 0)
 		(layer "F.SilkS")
@@
 		)
 	)
-	(gr_text "12V"
+	(gr_text "+12V"
 		(at 124.5 65.5 0)
 		(layer "F.SilkS")
@@
 		)
 	)
-	(gr_text "12V"
+	(gr_text "+12V"
 		(at 43.5 65.5 0)
 		(layer "F.SilkS")
@@
 		)
 	)
-	(gr_text "12V"
+	(gr_text "+12V"
 		(at 57 65.5 0)
 		(layer "F.SilkS")
@@
 		)
 	)
-	(gr_text "12V"
+	(gr_text "+12V"
 		(at 111 65.5 0)
 		(layer "F.SilkS")
