File: hardware/mtu-connection-board-large/locker-lg.kicad_pcb (KiCad board)
At the start: 2 copper layers, 175 x 90 mm, 32 parts

Commit message: style(pcb): clarify 12V silkscreen polarity
Co-authored-by: Cursor <cursoragent@cursor.com>
Other:
- board text added: "+12V"
- board text removed: "12V"
Changed lines of the file:
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@@
 		)
 	)
-	(gr_text "12V"
+	(gr_text "+12V"
 		(at 200 94.2895 0)
 		(layer "F.SilkS")
@@
 		)
 	)
-	(gr_text "12V"
+	(gr_text "+12V"
 		(at 159.5 94.2895 0)
 		(layer "F.SilkS")
@@
 		)
 	)
-	(gr_text "12V"
+	(gr_text "+12V"
 		(at 139 94.2895 0)
 		(layer "F.SilkS")
@@
 		)
 	)
-	(gr_text "12V"
+	(gr_text "+12V"
 		(at 104.5 135.5 270)
 		(layer "F.SilkS")
@@
 		)
 	)
-	(gr_text "12V"
+	(gr_text "+12V"
 		(at 139 135.5 270)
 		(layer "F.SilkS")
@@
 		)
 	)
-	(gr_text "12V"
+	(gr_text "+12V"
 		(at 210.5 94.2895 0)
 		(layer "F.SilkS")
@@
 		)
 	)
-	(gr_text "12V"
+	(gr_text "+12V"
 		(at 69.5 135.5 270)
 		(layer "F.SilkS")
@@
 		)
 	)
-	(gr_text "12V"
+	(gr_text "+12V"
 		(at 124 135.5 270)
 		(layer "F.SilkS")
@@
 		)
 	)
-	(gr_text "12V"
+	(gr_text "+12V"
 		(at 169.5 94.2895 0)
 		(layer "F.SilkS")
@@
 		)
 	)
-	(gr_text "12V"
+	(gr_text "+12V"
 		(at 190 94.2895 0)
 		(layer "F.SilkS")
@@
 		)
 	)
-	(gr_text "12V"
+	(gr_text "+12V"
 		(at 149 94.2895 0)
 		(layer "F.SilkS")
@@
 		)
 	)
-	(gr_text "12V"
+	(gr_text "+12V"
 		(at 84 135.5 270)
 		(layer "F.SilkS")
@@
 		)
 	)
-	(gr_text "12V"
+	(gr_text "+12V"
 		(at 179.5 94.2895 0)
 		(layer "F.SilkS")
